Commit message: ros framework fork for heal

File: cobot_ros2/addverb_cobot_description/urdf/heal.urdf (robot description, URDF)
Before this commit: robot robot, 16 links, 15 joints
Links:
- link base_link: mass 3.729 -> 5.0617
- link end-effector: mass 0.051095 -> 3.0617
- link link1: mass 7.919 -> 5.0617
- link link2: mass 1.017 -> 1.2353
- link link3: mass 5.574 -> 3.5577
- link link4: mass 1.894 -> 1.31
- link link5: mass 1.791 -> 1.1965
Joints:
- joint joint2: axis 1 0 0 -> -1 0 0; limit lower=-2.05 upper=0.75 effort=150 velocity=1 -> lower=-0.75 upper=2.05 effort=150 velocity=1
- joint joint3: axis -1 0 0 -> 1 0 0
- joint joint4: axis 0 1 0 -> 0 -1 0
- joint joint5: axis -0.5 0.86603 0 -> 0.5 0.86603 0

File: cobot_ros2/addverb_cobot_description/urdf/heal.urdf.xacro (robot description, xacro)
@@ -26,16 +26,8 @@
   <link name="link1">
     <inertial>
-      <origin
-        xyz="0.01254 0 0.272"
-        rpy="0 0 0" />
-      <mass
-        value="7.919" />
-      <inertia
-        ixx="0.044879950"
-        ixy="-7.346E-06"
-        ixz="-0.006377064"
-        iyy="0.047389946"
-        iyz="-1.534E-06"
-        izz="0.015930027" />
+      <origin xyz="-0.012435 -2.5345E-05 0.28172" rpy="0 0 0" />
+      <mass value="5.0617" />
+      <inertia ixx="0.011934" ixy="-4.2772E-06" ixz="0.0016521" iyy="0.011427" iyz="3.2849E-06"
+        izz="0.0091785" />
     </inertial>
     <visual>
@@ -64,16 +56,8 @@
   <link name="link2">
     <inertial>
-      <origin
-        xyz="0.10537 0 0.14998"
-        rpy="0 0 0" />
-      <mass
-        value="1.017" />
-      <inertia
-        ixx="0.016383576"
-        ixy="0"
-        ixz="5.01E-07"
-        iyy="0.015505423"
-        iyz="8.3217E-06"
-        izz="0.001453264" />
+      <origin xyz="-0.10679 3.7919E-06 0.15236" rpy="0 0 0" />
+      <mass value="1.2353" />
+      <inertia ixx="0.0057954" ixy="3.2114E-08" ixz="3.5658E-06" iyy="0.0048706" iyz="-6.4438E-07"
+        izz="0.0016259" />
     </inertial>
     <visual>
@@ -97,21 +81,13 @@
     <parent link="link1" />
     <child link="link2" />
-    <axis xyz="1 0 0" />
-    <limit lower="-2.05" upper="0.75" effort="150" velocity="1" />
+    <axis xyz="-1 0 0" />
+    <limit lower="-0.75" upper="2.05" effort="150" velocity="1" />
   </joint>
   <link name="link3">
     <inertial>
-      <origin
-        xyz="0.01755 0.03359 0"
-        rpy="0 0 0" />
-      <mass
-        value="5.574" />
-      <inertia
-        ixx="0.021340532"
-        ixy="0.003304844"
-        ixz="-1.2974E-06"
-        iyy="0.009841027"
-        iyz="1.3202E-05"
-        izz="0.023306443" />
+      <origin xyz="-0.017248 0.035025 -2.2087E-05" rpy="0 0 0" />
+      <mass value="3.5577" />
+      <inertia ixx="0.0066247" ixy="-0.00095453" ixz="1.793E-06" iyy="0.0050017" iyz="1.7882E-06"
+        izz="0.0060636" />
     </inertial>
     <visual>
@@ -135,21 +111,13 @@
     <parent link="link2" />
     <child link="link3" />
-    <axis xyz="-1 0 0" />
+    <axis xyz="1 0 0" />
     <limit lower="-1" upper="1" effort="150" velocity="5" />
   </joint>
   <link name="link4">
     <inertial>
-      <origin
-        xyz="0.05065 -0.1059 0"
-        rpy="0 0 0" />
-      <mass
-        value="1.894" />
-      <inertia
-        ixx="0.003626317"
-        ixy="-0.000600942"
-        ixz="2.750E-06"
-        iyy="0.002331370"
-        iyz="3.309E-06"
-        izz="0.004130374" />
+      <origin xyz="-0.047999 -0.10939 4.4809E-05" rpy="0 0 0" />
+      <mass value="1.31" />
+      <inertia ixx="0.0014749" ixy="0.00050231" ixz="1.7564E-06" iyy="0.0016894" iyz="-1.9993E-06"
+        izz="0.0017778" />
     </inertial>
     <visual>
@@ -178,16 +146,8 @@
   <link name="link5">
     <inertial>
-      <origin
-        xyz="0.00216 -0.00360 -0.04603"
-        rpy="0 0 0" />
-      <mass
-        value="1.791" />
-      <inertia
-        ixx="0.002516338"
-        ixy="6.5634E-05"
-        ixz="-0.000102333"
-        iyy="0.002442610"
-        iyz="0.000185747"
-        izz="0.001857540" />
+      <origin xyz="-0.0015193 -0.0027725 -0.044032" rpy="0 0 0" />
+      <mass value="1.1965" />
+      <inertia ixx="0.0010777" ixy="-3.7989E-05" ixz="2.9305E-05" iyy="0.0010311" iyz="4.9507E-05"
+        izz="0.0013412" />
     </inertial>
     <visual>
@@ -211,5 +171,5 @@
     <parent link="link4" />
     <child link="link5" />
-    <axis xyz="-0.5 0.86603 0" />
+    <axis xyz="0.5 0.86603 0" />
     <limit lower="-${pi}" upper="${pi}" effort="80" velocity="1" />
   </joint>

Commit message: updated urdf

File: cobot_ros2/addverb_cobot_description/urdf/heal.urdf (robot description, URDF)
Before this commit: robot robot, 16 links, 15 joints
Links:
- link base_link: mass 5.0617 -> 3.729
- link end-effector: mass 3.0617 -> 0.051095
- link link1: mass 5.0617 -> 7.919
- link link2: mass 1.2353 -> 1.017
- link link3: mass 3.5577 -> 5.574
- link link4: mass 1.31 -> 1.894
- link link5: mass 1.1965 -> 1.791

File: cobot_ros2/addverb_cobot_description/urdf/heal.urdf.xacro (robot description, xacro)
@@ -1,224 +1,105 @@
-<?xml version="1.0" encoding="utf-8"?>
-<robot xmlns:xacro="http://www.ros.org/wiki/xacro" name="robot">
-  <!--
-  This URDF was automatically created by SolidWorks to URDF Exporter! Originally created by Stephen
-  Brawner (brawner@gmail.com)
-     Commit Version: 1.6.0-4-g7f85cfe  Build Version: 1.6.7995.38578
-     For more information, please see http://wiki.ros.org/sw_urdf_exporter
-  -->
-  <link name="base_link">
-    <visual>
-      <origin xyz="0 0 0" rpy="0 0 0" />
-      <geometry>
-        <mesh filename="package://addverb_cobot_description/meshes/base_link.STL" />
-      </geometry>
-      <material name="">
-        <color rgba="0.75294 0.75294 0.75294 1" />
-      </material>
-    </visual>
-    <collision>
-      <origin xyz="0 0 0" rpy="0 0 0" />
-      <geometry>
-        <mesh filename="package://addverb_cobot_description/meshes/base_link.STL" />
-      </geometry>
-    </collision>
-  </link>
-  <link name="link1">
-    <inertial>
-      <origin xyz="-0.012435 -2.5345E-05 0.28172" rpy="0 0 0" />
-      <mass value="5.0617" />
-      <inertia ixx="0.011934" ixy="-4.2772E-06" ixz="0.0016521" iyy="0.011427" iyz="3.2849E-06"
-        izz="0.0091785" />
-    </inertial>
-    <visual>
-      <origin xyz="0 0 0" rpy="0 0 0" />
-      <geometry>
-        <mesh filename="package://addverb_cobot_description/meshes/link1.STL" />
-      </geometry>
-      <material name="">
-        <color rgba="0.75294 0.75294 0.75294 1" />
-      </material>
-    </visual>
-    <collision>
-      <origin xyz="0 0 0" rpy="0 0 0" />
-      <geometry>
-        <mesh filename="package://addverb_cobot_description/meshes/link1.STL" />
-      </geometry>
-    </collision>
-  </link>
-  <joint name="joint1" type="revolute">
-    <origin xyz="0 0 0" rpy="0 0 0" />
-    <parent link="base_link" />
-    <child link="link1" />
-    <axis xyz="0 0 1" />
-    <limit lower="-${pi}" upper="${pi}" effort="150" velocity="3" />
-  </joint>
-  <link name="link2">
-    <inertial>
-      <origin xyz="-0.10679 3.7919E-06 0.15236" rpy="0 0 0" />
-      <mass value="1.2353" />
-      <inertia ixx="0.0057954" ixy="3.2114E-08" ixz="3.5658E-06" iyy="0.0048706" iyz="-6.4438E-07"
-        izz="0.0016259" />
-    </inertial>
-    <visual>
-      <origin xyz="0 0 0" rpy="0 0 0" />
-      <geometry>
-        <mesh filename="package://addverb_cobot_description/meshes/link2.STL" />
-      </geometry>
-      <material name="">
-        <color rgba="0.75294 0.75294 0.75294 1" />
-      </material>
-    </visual>
-    <collision>
-      <origin xyz="0 0 0" rpy="0 0 0" />
-      <geometry>
-        <mesh filename="package://addverb_cobot_description/meshes/link2.STL" />
-      </geometry>
-    </collision>
-  </link>
-  <joint name="joint2" type="revolute">
-    <origin xyz="0 0 0.346" rpy="0 0 0" />
-    <parent link="link1" />
-    <child link="link2" />
-    <axis xyz="-1 0 0" />
-    <limit lower="-0.75" upper="2.05" effort="150" velocity="1" />
-  </joint>
-  <link name="link3">
-    <inertial>
-      <origin xyz="-0.017248 0.035025 -2.2087E-05" rpy="0 0 0" />
-      <mass value="3.5577" />
-      <inertia ixx="0.0066247" ixy="-0.00095453" ixz="1.793E-06" iyy="0.0050017" iyz="1.7882E-06"
-        izz="0.0060636" />
-    </inertial>
-    <visual>
-      <origin xyz="0 0 0" rpy="0 0 0" />
-      <geometry>
-        <mesh filename="package://addverb_cobot_description/meshes/link3.STL" />
-      </geometry>
-      <material name="">
-        <color rgba="0.75294 0.75294 0.75294 1" />
-      </material>
-    </visual>
-    <collision>
-      <origin xyz="0 0 0" rpy="0 0 0" />
-      <geometry>
-        <mesh filename="package://addverb_cobot_description/meshes/link3.STL" />
-      </geometry>
-    </collision>
-  </link>
-  <joint name="joint3" type="revolute">
-    <origin xyz="0 0 0.305" rpy="0 0 0" />
-    <parent link="link2" />
-    <child link="link3" />
-    <axis xyz="1 0 0" />
-    <limit lower="-1" upper="1" effort="150" velocity="5" />
-  </joint>
-  <link name="link4">
-    <inertial>
-      <origin xyz="-0.047999 -0.10939 4.4809E-05" rpy="0 0 0" />
-      <mass value="1.31" />
-      <inertia ixx="0.0014749" ixy="0.00050231" ixz="1.7564E-06" iyy="0.0016894" iyz="-1.9993E-06"
-        izz="0.0017778" />
-    </inertial>
-    <visual>
-      <origin xyz="0 0 0" rpy="0 0 0" />
-      <geometry>
-        <mesh filename="package://addverb_cobot_description/meshes/link4.STL" />
-      </geometry>
-      <material name="">
-        <color rgba="0.75294 0.75294 0.75294 1" />
-      </material>
-    </visual>
-    <collision>
-      <origin xyz="0 0 0" rpy="0 0 0" />
-      <geometry>
-        <mesh filename="package://addverb_cobot_description/meshes/link4.STL" />
-      </geometry>
-    </collision>
-  </link>
-  <joint name="joint4" type="revolute">
-    <origin xyz="-0.0009127 0.36813 0" rpy="0 0 0" />
-    <parent link="link3" />
-    <child link="link4" />
-    <axis xyz="0 1 0" />
-    <limit lower="-${pi}" upper="${pi}" effort="80" velocity="1" />
-  </joint>
-  <link name="link5">
-    <inertial>
-      <origin xyz="-0.0015193 -0.0027725 -0.044032" rpy="0 0 0" />
-      <mass value="1.1965" />
-      <inertia ixx="0.0010777" ixy="-3.7989E-05" ixz="2.9305E-05" iyy="0.0010311" iyz="4.9507E-05"
-        izz="0.0013412" />
-    </inertial>
-    <visual>
-      <origin xyz="0 0 0" rpy="0 0 0" />
-      <geometry>
-        <mesh filename="package://addverb_cobot_description/meshes/link5.STL" />
-      </geometry>
-      <material name="">
-        <color rgba="0.75294 0.75294 0.75294 1" />
-      </material>
-    </visual>
-    <collision>
-      <origin xyz="0 0 0" rpy="0 0 0" />
-      <geometry>
-        <mesh filename="package://addverb_cobot_description/meshes/link5.STL" />
-      </geometry>
-    </collision>
-  </link>
-  <joint name="joint5" type="revolute">
-    <origin xyz="0 0 0" rpy="0 0 0" />
-    <parent link="link4" />
-    <child link="link5" />
-    <axis xyz="0.5 0.86603 0" />
-    <limit lower="-${pi}" upper="${pi}" effort="80" velocity="1" />
-  </joint>
-  <link name="end-effector" />
+<?xml version="1.0"?>
+<robot xmlns:xacro="http://www.ros.org/wiki/xacro" name="cobot2">
+  <xacro:property name="pi" value="3.141592653589793"/>
+  <!-- ================= MACROS ================= -->
+  <xacro:macro name="cobot_link" params="name mesh mass xyz rpy ixx ixy ixz iyy iyz izz">
+    <link name="${name}">
+      <inertial>
+        <origin xyz="${xyz}" rpy="${rpy}"/>
+        <mass value="${mass}"/>
+        <inertia
+          ixx="${ixx}" ixy="${ixy}" ixz="${ixz}"
+          iyy="${iyy}" iyz="${iyz}" izz="${izz}"/>
+      </inertial>
+      <visual>
+        <origin xyz="0 0 0" rpy="0 0 0"/>
+        <geometry>
+          <mesh filename="package://addverb_cobot_description/meshes/${mesh}"/>
+        </geometry>
+      </visual>
+      <collision>
+        <origin xyz="0 0 0" rpy="0 0 0"/>
+        <geometry>
+          <mesh filename="package://addverb_cobot_description/meshes/${mesh}"/>
+        </geometry>
+      </collision>
+    </link>
+  </xacro:macro>
+  <xacro:macro name="cobot_joint" params="name parent child xyz rpy axis lower upper effort velocity">
+    <joint name="${name}" type="revolute">
+      <origin xyz="${xyz}" rpy="${rpy}"/>
+      <parent link="${parent}"/>
+      <child link="${child}"/>
+      <axis xyz="${axis}"/>
+      <limit lower="${lower}" upper="${upper}" effort="${effort}" velocity="${velocity}"/>
+    </joint>
+  </xacro:macro>
+  <!-- ================= ARM ================= -->
+  <xacro:cobot_link name="base_link" mesh="base_link.STL"
+    mass="3.729" xyz="0 0 0.019" rpy="0 0 0"
+    ixx="0.016307106" ixy="2.079E-06" ixz="-1.378E-06"
+    iyy="0.016302834" iyz="-4.998E-06" izz="0.022458155"/>
+  <xacro:cobot_link name="link1" mesh="link1.STL"
+    mass="7.919" xyz="-0.01254 0 0.272" rpy="0 0 0"
+    ixx="0.044879950" ixy="7.346E-06" ixz="0.006377064"
+    iyy="0.047389946" iyz="-1.534E-06" izz="0.015930027"/>
+  <xacro:cobot_link name="link2" mesh="link2.STL"
+    mass="1.017" xyz="-0.10537 0 0.14998" rpy="0 0 0"
+    ixx="0.016383576" ixy="0" ixz="-5.01E-07"
+    iyy="0.015505423" iyz="8.3217E-06" izz="0.001453264"/>
+  <xacro:cobot_link name="link3" mesh="link3.STL"
+    mass="5.574" xyz="-0.01755 0.03359 0" rpy="0 0 0"
+    ixx="0.021340532" ixy="-0.003304844" ixz="1.2974E-06"
+    iyy="0.009841027" iyz="1.3202E-05" izz="0.023306443"/>
+  <xacro:cobot_link name="link4" mesh="link4.STL"
+    mass="1.894" xyz="-0.05065 -0.1059 0" rpy="0 0 0"
+    ixx="0.003626317" ixy="0.000600942" ixz="-2.750E-06"
+    iyy="0.002331370" iyz="3.309E-06" izz="0.004130374"/>
+  <xacro:cobot_link name="link5" mesh="link5.STL"
+    mass="1.791" xyz="-0.00216 -0.00360 -0.04603" rpy="0 0 0"
+    ixx="0.002516338" ixy="-6.5634E-05" ixz="0.000102333"
+    iyy="0.002442610" iyz="0.000185747" izz="0.001857540"/>
+  <!-- JOINTS -->
+  <xacro:cobot_joint name="joint1" parent="base_link" child="link1"
+    xyz="0 0 0" rpy="0 0 0" axis="0 0 1"
+    lower="-${pi}" upper="${pi}" effort="150" velocity="3"/>
+  <xacro:cobot_joint name="joint2" parent="link1" child="link2"
+    xyz="0 0 0.346" rpy="0 0 0" axis="-1 0 0"
+    lower="-0.75" upper="2.05" effort="150" velocity="1"/>
+  <xacro:cobot_joint name="joint3" parent="link2" child="link3"
+    xyz="0 0 0.305" rpy="0 0 0" axis="1 0 0"
+    lower="-1" upper="1" effort="150" velocity="5"/>
+  <xacro:cobot_joint name="joint4" parent="link3" child="link4"
+    xyz="-0.0009127 0.36813 0" rpy="0 0 0" axis="0 -1 0"
+    lower="-${pi}" upper="${pi}" effort="80" velocity="1"/>
+  <xacro:cobot_joint name="joint5" parent="link4" child="link5"
+    xyz="0 0 0" rpy="0 0 0" axis="0.5 0.86603 0"
+    lower="-${pi}" upper="${pi}" effort="80" velocity="1"/>
+  <!-- ================= END EFFECTOR ================= -->
+  <link name="end-effector">
+    <inertial>
+      <origin xyz="0 0 -0.0014" rpy="0 0 0"/>
+      <mass value="0.051095"/>
+      <inertia ixx="2.8814E-05" ixy="0" ixz="0"
+               iyy="2.8814E-05" iyz="0" izz="5.7263E-05"/>
+    </inertial>
+  </link>
   <joint name="joint6" type="revolute">
-    <origin xyz="0 0 -0.0975" rpy="0 0 0" />
-    <parent link="link5" />
-    <child link="end-effector" />
-    <axis xyz="0 0 -1" />
-    <limit lower="-${pi}" upper="${pi}" effort="80" velocity="1" />
-  </joint>
-  <link
-    name="robotiq_85_base_link">
-    <inertial>
-      <origin
-        xyz="0.00021987 -2.3546E-10 0.030163"
-        rpy="0 0 0" />
-      <mass
-        value="0.30915" />
-      <inertia
-        ixx="0.00028972"
-        ixy="-5.7879E-10"
-        ixz="-1.8543E-06"
-        iyy="0.00030737"
-        iyz="1.682E-12"
-        izz="0.00019914" />
-    </inertial>
-    <visual>
-      <origin
-        xyz="0 0 0"
-        rpy="0 0 0" />
-      <geometry>
-        <mesh
-          filename="package://addverb_cobot_description/meshes/robotiq_85_base_link_fine.STL" />
-      </geometry>
-      <material
-        name="">
-        <color
-          rgba="0.1 0.1 0.1 1" />
-      </material>
-    </visual>
-    <collision>
-      <origin
-        xyz="0 0 0"
-        rpy="0 0 0" />
-      <geometry>
-        <mesh
-          filename="package://addverb_cobot_description/meshes/robotiq_85_base_link_coarse.STL" />
-      </geometry>
-    </collision>
+    <origin xyz="0 0 -0.0975" rpy="0 0 0"/>
+    <parent link="link5"/>
+    <child link="end-effector"/>
+    <axis xyz="0 0 -1"/>
+    <limit lower="-${pi}" upper="${pi}" effort="80" velocity="1"/>
+  </joint>
+  <!-- ================= GRIPPER (UNCHANGED) ================= -->
+  <!-- Paste EXACTLY as-is below (no macros) -->
+  <!-- robotiq base -->
+  <link name="robotiq_85_base_link">
+    <inertial>
+      <origin xyz="0.00021987 -2.3546E-10 0.030163"/>
+      <mass value="0.30915"/>
+      <inertia ixx="0.00028972" ixy="-5.7879E-10" ixz="-1.8543E-06"
+               iyy="0.00030737" iyz="1.682E-12" izz="0.00019914"/>
+    </inertial>
   </link>
   <joint name="joint7" type="fixed">
@@ -227,12 +108,8 @@
     <child link="robotiq_85_base_link"/>
   </joint>
-  <link
-    name="left_outer_knuckle">
-    <inertial>
-      <origin
-        xyz="0.0178331863169983 3.68915177224286E-11 0.0021442477325704"
-        rpy="0 0 0" />
-      <mass
-        value="0.00684838849434396" />
+  <link name="left_outer_knuckle">
+    <inertial>
+      <origin xyz="0.0178331863169983 3.68915177224286E-11 0.0021442477325704" rpy="0 0 0"/>
+      <mass value="0.00684838849434396"/>
       <inertia
         ixx="2.66832029033166E-07"
@@ -241,56 +118,33 @@
         iyy="1.3889233257419E-06"
         iyz="2.82951161241588E-15"
-        izz="1.26603336914415E-06" />
-    </inertial>
-    <visual>
-      <origin
-        xyz="0 0 0"
-        rpy="0 0 0" />
-      <geometry>
-        <mesh
-          filename="package://addverb_cobot_description/meshes/outer_knuckle_fine.STL" />
-      </geometry>
-      <material
-        name="">
-        <color
-          rgba="0.1 0.1 0.1 1" />
-      </material>
-    </visual>
-    <collision>
-      <origin
-        xyz="0 0 0"
-        rpy="0 0 0" />
-      <geometry>
-        <mesh
-          filename="package://addverb_cobot_description/meshes/outer_knuckle_coarse.STL" />
-      </geometry>
-    </collision>
-  </link>
-  <joint
-    name="finger_joint"
-    type="revolute">
-    <origin
-      xyz="0.0306011444260539 0 0.0627920162695395"
-      rpy="0 0 0" />
-    <parent
-      link="robotiq_85_base_link" />
-    <child
-      link="left_outer_knuckle" />
-    <axis
-      xyz="0 -1 0" />
-    <limit
-	  lower="0"
-      upper="0.725"
-      velocity="2.0"
-      effort="1000" />
-  </joint>
-  <link
-    name="left_outer_finger">
-    <inertial>
-      <origin
-        xyz="0.00131451599174296 2.88942057994543E-15 0.0215404163180413"
-        rpy="0 0 0" />
-      <mass
-        value="0.0273093985570947" />
+        izz="1.26603336914415E-06"/>
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