Commit message: updated moveit config, added dockerfil : syncro_ros2 script

File: cobot_ros2/addverb_cobot_description/urdf/heal.urdf.xacro (robot description, xacro)
@@ -11,5 +11,5 @@
       <origin xyz="0 0 0" rpy="0 0 0" />
       <geometry>
-        <mesh filename="package://addverb_cobot_description/meshes/base_link.STL" />
+        <mesh filename="package://addverb_cobot_description/heal_meshes/base_link.STL" />
       </geometry>
       <material name="">
@@ -20,5 +20,5 @@
       <origin xyz="0 0 0" rpy="0 0 0" />
       <geometry>
-        <mesh filename="package://addverb_cobot_description/meshes/base_link.STL" />
+        <mesh filename="package://addverb_cobot_description/heal_meshes/base_link.STL" />
       </geometry>
     </collision>
@@ -42,5 +42,5 @@
       <origin xyz="0 0 0" rpy="0 0 0" />
       <geometry>
-        <mesh filename="package://addverb_cobot_description/meshes/link1.STL" />
+        <mesh filename="package://addverb_cobot_description/heal_meshes/link1.STL" />
       </geometry>
       <material name="">
@@ -51,5 +51,5 @@
       <origin xyz="0 0 0" rpy="0 0 0" />
       <geometry>
-        <mesh filename="package://addverb_cobot_description/meshes/link1.STL" />
+        <mesh filename="package://addverb_cobot_description/heal_meshes/link1.STL" />
       </geometry>
     </collision>
@@ -80,5 +80,5 @@
       <origin xyz="0 0 0" rpy="0 0 0" />
       <geometry>
-        <mesh filename="package://addverb_cobot_description/meshes/link2.STL" />
+        <mesh filename="package://addverb_cobot_description/heal_meshes/link2.STL" />
       </geometry>
       <material name="">
@@ -89,5 +89,5 @@
       <origin xyz="0 0 0" rpy="0 0 0" />
       <geometry>
-        <mesh filename="package://addverb_cobot_description/meshes/link2.STL" />
+        <mesh filename="package://addverb_cobot_description/heal_meshes/link2.STL" />
       </geometry>
     </collision>
@@ -118,5 +118,5 @@
       <origin xyz="0 0 0" rpy="0 0 0" />
       <geometry>
-        <mesh filename="package://addverb_cobot_description/meshes/link3.STL" />
+        <mesh filename="package://addverb_cobot_description/heal_meshes/link3.STL" />
       </geometry>
       <material name="">
@@ -127,5 +127,5 @@
       <origin xyz="0 0 0" rpy="0 0 0" />
       <geometry>
-        <mesh filename="package://addverb_cobot_description/meshes/link3.STL" />
+        <mesh filename="package://addverb_cobot_description/heal_meshes/link3.STL" />
       </geometry>
     </collision>
@@ -156,5 +156,5 @@
       <origin xyz="0 0 0" rpy="0 0 0" />
       <geometry>
-        <mesh filename="package://addverb_cobot_description/meshes/link4.STL" />
+        <mesh filename="package://addverb_cobot_description/heal_meshes/link4.STL" />
       </geometry>
       <material name="">
@@ -165,5 +165,5 @@
       <origin xyz="0 0 0" rpy="0 0 0" />
       <geometry>
-        <mesh filename="package://addverb_cobot_description/meshes/link4.STL" />
+        <mesh filename="package://addverb_cobot_description/heal_meshes/link4.STL" />
       </geometry>
     </collision>
@@ -194,5 +194,5 @@
       <origin xyz="0 0 0" rpy="0 0 0" />
       <geometry>
-        <mesh filename="package://addverb_cobot_description/meshes/link5.STL" />
+        <mesh filename="package://addverb_cobot_description/heal_meshes/link5.STL" />
       </geometry>
       <material name="">
@@ -203,5 +203,5 @@
       <origin xyz="0 0 0" rpy="0 0 0" />
       <geometry>
-        <mesh filename="package://addverb_cobot_description/meshes/link5.STL" />
+        <mesh filename="package://addverb_cobot_description/heal_meshes/link5.STL" />
       </geometry>
     </collision>
@@ -244,19 +244,19 @@
       <geometry>
         <mesh
-          filename="package://addverb_cobot_description/meshes/robotiq_85_base_link_fine.STL" />
-      </geometry>
-      <material
-        name="">
-        <color
-          rgba="0.1 0.1 0.1 1" />
-      </material>
-    </visual>
-    <collision>
-      <origin
-        xyz="0 0 0"
-        rpy="0 0 0" />
-      <geometry>
-        <mesh
-          filename="package://addverb_cobot_description/meshes/robotiq_85_base_link_coarse.STL" />
+          filename="package://addverb_cobot_description/heal_meshes/robotiq_85_base_link_fine.STL" />
+      </geometry>
+      <material
+        name="">
+        <color
+          rgba="0.1 0.1 0.1 1" />
+      </material>
+    </visual>
+    <collision>
+      <origin
+        xyz="0 0 0"
+        rpy="0 0 0" />
+      <geometry>
+        <mesh
+          filename="package://addverb_cobot_description/heal_meshes/robotiq_85_base_link_coarse.STL" />
       </geometry>
     </collision>
@@ -289,19 +289,19 @@
       <geometry>
         <mesh
-          filename="package://addverb_cobot_description/meshes/outer_knuckle_fine.STL" />
-      </geometry>
-      <material
-        name="">
-        <color
-          rgba="0.1 0.1 0.1 1" />
-      </material>
-    </visual>
-    <collision>
-      <origin
-        xyz="0 0 0"
-        rpy="0 0 0" />
-      <geometry>
-        <mesh
-          filename="package://addverb_cobot_description/meshes/outer_knuckle_coarse.STL" />
+          filename="package://addverb_cobot_description/heal_meshes/outer_knuckle_fine.STL" />
+      </geometry>
+      <material
+        name="">
+        <color
+          rgba="0.1 0.1 0.1 1" />
+      </material>
+    </visual>
+    <collision>
+      <origin
+        xyz="0 0 0"
+        rpy="0 0 0" />
+      <geometry>
+        <mesh
+          filename="package://addverb_cobot_description/heal_meshes/outer_knuckle_coarse.STL" />
       </geometry>
     </collision>
@@ -347,19 +347,19 @@
       <geometry>
         <mesh
-          filename="package://addverb_cobot_description/meshes/outer_finger_fine.STL" />
-      </geometry>
-      <material
-        name="">
-        <color
-          rgba="0.1 0.1 0.1 1" />
-      </material>
-    </visual>
-    <collision>
-      <origin
-        xyz="0 0 0"
-        rpy="0 0 0" />
-      <geometry>
-        <mesh
-          filename="package://addverb_cobot_description/meshes/outer_finger_coarse.STL" />
+          filename="package://addverb_cobot_description/heal_meshes/outer_finger_fine.STL" />
+      </geometry>
+      <material
+        name="">
+        <color
+          rgba="0.1 0.1 0.1 1" />
+      </material>
+    </visual>
+    <collision>
+      <origin
+        xyz="0 0 0"
+        rpy="0 0 0" />
+      <geometry>
+        <mesh
+          filename="package://addverb_cobot_description/heal_meshes/outer_finger_coarse.STL" />
       </geometry>
     </collision>
@@ -400,19 +400,19 @@
       <geometry>
         <mesh
-          filename="package://addverb_cobot_description/meshes/inner_knuckle_fine.STL" />
-      </geometry>
-      <material
-        name="">
-        <color
-          rgba="0.1 0.1 0.1 1" />
-      </material>
-    </visual>
-    <collision>
-      <origin
-        xyz="0 0 0"
-        rpy="0 0 0" />
-      <geometry>
-        <mesh
-          filename="package://addverb_cobot_description/meshes/inner_knuckle_coarse.STL" />
+          filename="package://addverb_cobot_description/heal_meshes/inner_knuckle_fine.STL" />
+      </geometry>
+      <material
+        name="">
+        <color
+          rgba="0.1 0.1 0.1 1" />
+      </material>
+    </visual>
+    <collision>
+      <origin
+        xyz="0 0 0"
+        rpy="0 0 0" />
+      <geometry>
+        <mesh
+          filename="package://addverb_cobot_description/heal_meshes/inner_knuckle_coarse.STL" />
       </geometry>
     </collision>
@@ -462,19 +462,19 @@
       <geometry>
         <mesh
-          filename="package://addverb_cobot_description/meshes/inner_finger_fine.STL" />
-      </geometry>
-      <material
-        name="">
-        <color
-          rgba="0.1 0.1 0.1 1" />
-      </material>
-    </visual>
-    <collision>
-      <origin
-        xyz="0 0 0"
-        rpy="0 0 0" />
-      <geometry>
-        <mesh
-          filename="package://addverb_cobot_description/meshes/inner_finger_coarse.STL" />
+          filename="package://addverb_cobot_description/heal_meshes/inner_finger_fine.STL" />
+      </geometry>
+      <material
+        name="">
+        <color
+          rgba="0.1 0.1 0.1 1" />
+      </material>
+    </visual>
+    <collision>
+      <origin
+        xyz="0 0 0"
+        rpy="0 0 0" />
+      <geometry>
+        <mesh
+          filename="package://addverb_cobot_description/heal_meshes/inner_finger_coarse.STL" />
       </geometry>
     </collision>
@@ -524,19 +524,19 @@
       <geometry>
         <mesh
-          filename="package://addverb_cobot_description/meshes/inner_knuckle_fine.STL" />
-      </geometry>
-      <material
-        name="">
-        <color
-          rgba="0.1 0.1 0.1 1" />
-      </material>
-    </visual>
-    <collision>
-      <origin
-        xyz="0 0 0"
-        rpy="0 0 0" />
-      <geometry>
-        <mesh
-          filename="package://addverb_cobot_description/meshes/inner_knuckle_coarse.STL" />
+          filename="package://addverb_cobot_description/heal_meshes/inner_knuckle_fine.STL" />
+      </geometry>
+      <material
+        name="">
+        <color
+          rgba="0.1 0.1 0.1 1" />
+      </material>
+    </visual>
+    <collision>
+      <origin
+        xyz="0 0 0"
+        rpy="0 0 0" />
+      <geometry>
+        <mesh
+          filename="package://addverb_cobot_description/heal_meshes/inner_knuckle_coarse.STL" />
       </geometry>
     </collision>
@@ -586,19 +586,19 @@
       <geometry>
         <mesh
-          filename="package://addverb_cobot_description/meshes/inner_finger_fine.STL" />
-      </geometry>
-      <material
-        name="">
-        <color
-          rgba="0.1 0.1 0.1 1" />
-      </material>
-    </visual>
-    <collision>
-      <origin
-        xyz="0 0 0"
-        rpy="0 0 0" />
-      <geometry>
-        <mesh
-          filename="package://addverb_cobot_description/meshes/inner_finger_coarse.STL" />
+          filename="package://addverb_cobot_description/heal_meshes/inner_finger_fine.STL" />
+      </geometry>
+      <material
+        name="">
+        <color
+          rgba="0.1 0.1 0.1 1" />
+      </material>
+    </visual>
+    <collision>
+      <origin
+        xyz="0 0 0"
+        rpy="0 0 0" />
+      <geometry>
+        <mesh
+          filename="package://addverb_cobot_description/heal_meshes/inner_finger_coarse.STL" />
       </geometry>
     </collision>
@@ -648,19 +648,19 @@
       <geometry>
         <mesh
-          filename="package://addverb_cobot_description/meshes/outer_knuckle_fine.STL" />
-      </geometry>
-      <material
-        name="">
-        <color
-          rgba="0.1 0.1 0.1 1" />
-      </material>
-    </visual>
-    <collision>
-      <origin
-        xyz="0 0 0"
-        rpy="0 0 0" />
-      <geometry>
-        <mesh
-          filename="package://addverb_cobot_description/meshes/outer_knuckle_coarse.STL" />
+          filename="package://addverb_cobot_description/heal_meshes/outer_knuckle_fine.STL" />
+      </geometry>
+      <material
+        name="">
+        <color
+          rgba="0.1 0.1 0.1 1" />
+      </material>
+    </visual>
+    <collision>
+      <origin
+        xyz="0 0 0"
+        rpy="0 0 0" />
+      <geometry>
+        <mesh
+          filename="package://addverb_cobot_description/heal_meshes/outer_knuckle_coarse.STL" />
       </geometry>
     </collision>
@@ -710,19 +710,19 @@
       <geometry>
         <mesh
-          filename="package://addverb_cobot_description/meshes/outer_finger_fine.STL" />
-      </geometry>
-      <material
-        name="">
-        <color
-          rgba="0.1 0.1 0.1 1" />
-      </material>
-    </visual>
-    <collision>
-      <origin
-        xyz="0 0 0"
-        rpy="0 0 0" />
-      <geometry>
-        <mesh
-          filename="package://addverb_cobot_description/meshes/outer_finger_coarse.STL" />
+          filename="package://addverb_cobot_description/heal_meshes/outer_finger_fine.STL" />
+      </geometry>
+      <material
+        name="">
+        <color
+          rgba="0.1 0.1 0.1 1" />
+      </material>
+    </visual>
+    <collision>
+      <origin
+        xyz="0 0 0"
+        rpy="0 0 0" />
+      <geometry>
+        <mesh
+          filename="package://addverb_cobot_description/heal_meshes/outer_finger_coarse.STL" />
       </geometry>
     </collision>

File: cobot_ros2/addverb_cobot_description/urdf/syncro_ros2_control.urdf.xacro (robot description, xacro)
@@ -1,4 +1,4 @@
 <?xml version="1.0"?>
-<robot name="drdo_dual_arm" xmlns:xacro="http://www.ros.org/wiki/xacro">
+<robot name="robot" xmlns:xacro="http://www.ros.org/wiki/xacro">
   <xacro:include filename="$(find addverb_cobot_description)/urdf/syncro.urdf.xacro"/>
   <xacro:include filename="$(find addverb_cobot_description)/ros2_control/syncro.ros2_control.xacro"/>
